File: Project/plates/plate 625u.kicad_pcb (KiCad board)
At the start: 2 copper layers, 279.3 x 89.2 mm, 49 parts

Commit message: pcb & plate revisions
Other:
- outline, holes or cut-outs redrawn
- board text added: "V2 using cipu stabs for hopefully better result"
- board text removed: "one assembly on 625 is not usable"
