File: Project/plates/plate split 2u.kicad_pcb (KiCad board)
At the start: 2 copper layers, 279.3 x 89.2 mm, 52 parts

Commit message: fresh gerbers
Parts:
- removed the REF** at (167.5, 108.7)
- removed the REF** at (119.9, 108.7)
Other:
- outline, holes or cut-outs redrawn

Commit message: pcb & plate revisions
Other:
- outline, holes or cut-outs redrawn
- board text added: "V2 using cipu stabs for hopefully better result"
